Commit message: feat:updated robot description and drive controller

File: robo_car_description/urdf/ros_controllers.xacro (robot description, xacro)
@@ -18,5 +18,5 @@
             <robot_namespace>robo_car</robot_namespace>
             <robot_param_node>robot_state_publisher</robot_param_node>
-            <parameters>$(find robo_car_description)/config/controllers.yaml</parameters>
+            <parameters>$(find robo_car_description)/config/robo_car_controllers.yaml</parameters>
         </plugin>
     </gazebo>

File: robo_car_description/urdf/sensors/cam.xacro (robot description, xacro)
@@ -1,77 +1,78 @@
 <?xml version="1.0"?>
-<robot xmlns:xacro="http://www.ros.org/wiki/xacro"  name="robo_car">
-    <!-- <xacro:arg name="cam_visual"   default="false"/> -->
-    <!-- CAMERA LINK FRAME -->
-    <joint name="cam_joint" type="fixed">
-        <parent link="base_chassis_link"/>
-        <child link="cam_link"/>
-        <origin xyz="0.12 0 ${full_chassis_height}" rpy="0 0 0"/>
-    </joint>
-    <link name="cam_link">
-        <visual>
-            <origin xyz="-0.005 0 0" rpy="0 ${pi/2} 0"/>
-            <geometry>
-                <cylinder radius="0.01" length="0.01"/>
-            </geometry>
-            <material name="grey"/>
-        </visual>
-        <visual>
-            <origin xyz="-0.015 0 0" rpy="0 0 0"/>
-            <geometry>
-                <box size="0.01 0.04 0.025" />
-            </geometry>
-            <material name="grey"/>
-        </visual>
-        <collision>
-            <origin xyz="-0.01 0 0" rpy="0 0 0"/>
-            <geometry>
-                <box size="0.02 0.04 0.025"/>
-            </geometry>
-        </collision>
-        <xacro:inertial_box mass="0.0005" x="0.02" y="0.04" z="0.025">
-            <origin xyz="-0.01 0 0" rpy="0 0 0"/>
-        </xacro:inertial_box>
-    </link>
-    <joint name="cam_optical_joint" type="fixed">
-        <parent link="cam_link"/>
-        <child link="cam_optical_link"/>
-        <origin xyz="0 0 0" rpy="${-pi/2} 0 ${-pi/2}"/>
-    </joint>
-    <link name="cam_optical_link"/>
-    <gazebo reference="cam_link">
-        <material>Gazebo/DarkGrey</material>
-        <sensor type="camera" name="camera">
-            <visualize>$(arg cam_visual)</visualize>
-            <update_rate>15.0</update_rate>
-            <camera name="cam">
-                <horizontal_fov>1.4</horizontal_fov>
-                <image>
-                    <width>320</width>
-                    <height>240</height>
-                    <format>R8G8B8</format>
-                </image>
-                <clip>
-                    <near>0.05</near>
-                    <far>5</far>
-                </clip>
-                <noise>
-                    <type>gaussian</type>
-                    <mean>0.0</mean>
-                    <stddev>0.007</stddev>
-                </noise>
-            </camera>
-            <plugin name="rgb_cam_plugin" filename="libgazebo_ros_camera.so">
-                <!-- <ros>
-                    <namespace>cam</namespace>
-                    <remapping>~/image_raw:=raw</remapping>
-                    <remapping>~/camera_info:=info</remapping>
-                </ros> -->
-                <!-- Set camera name. If empty, defaults to sensor name (i.e. "sensor_name") -->
-                <camera_name>cam</camera_name>
-                <!-- Set TF frame name. If empty, defaults to link name (i.e. "link_name") -->
-                <frame_name>cam_optical_link</frame_name>
-                <hack_baseline>0.2</hack_baseline>
-            </plugin>
-        </sensor>
-    </gazebo>
+<robot xmlns:xacro="http://www.ros.org/wiki/xacro" >
+    <xacro:macro name="insert_camera" params="base_name parent_name x y z mass width height min_range max_range tilt_angle visualize">
+        <joint name="${base_name}_joint" type="fixed">
+            <parent link="${parent_name}"/>
+            <child link="${base_name}"/>
+            <origin xyz="${x} ${y} ${z}" rpy="0 ${tilt_angle} 0"/>
+        </joint>
+        <link name="${base_name}">
+            <visual>
+                <origin xyz="-0.02 0 0" rpy="0 ${-pi/2} 0"/>
+                <geometry>
+                    <cylinder radius="0.015" length="0.04"/>
+                </geometry>
+                <material name="grey"/>
+            </visual>
+            <visual>
+                <origin xyz="-0.03 0 0" rpy="0 ${-pi/2} 0"/>
+                <geometry>
+                    <!-- <cylinder radius="0.03" length="0.02"/> -->
+                    <box size="0.04 0.06 0.02"/>
+                </geometry>
+                <material name="grey"/>
+            </visual>
+            <collision>
+                <origin xyz="-0.02 0 0" rpy="0 ${-pi/2} 0"/>
+                <geometry>
+                    <cylinder radius="0.02" length="0.04"/>
+                </geometry>
+            </collision>
+            <xacro:inertial_cylinder mass="${mass}" radius="0.02" length="0.04">
+                <origin xyz="-0.02 0 0" rpy="0 ${-pi/2} 0"/>
+            </xacro:inertial_cylinder>
+        </link>
+        <joint name="${base_name}_optical_joint" type="fixed">
+            <parent link="${base_name}"/>
+            <child link="${base_name}_optical_link"/>
+            <origin xyz="0 0 0" rpy="${-pi/2} 0 ${-pi/2}"/>
+        </joint>
+        <link name="${base_name}_optical_link"/>
+        <gazebo reference="${base_name}">
+            <material>Gazebo/DarkGrey</material>
+            <sensor type="${base_name}" name="camera">
+                <visualize>${visualize}</visualize>
+                <update_rate>20.0</update_rate>
+                <camera name="${base_name}">
+                    <horizontal_fov>1.4</horizontal_fov>
+                    <image>
+                        <width>${width}</width>
+                        <height>${height}</height>
+                        <format>R8G8B8</format>
+                    </image>
+                    <clip>
+                        <near>${min_range}</near>
+                        <far>${max_range}</far>
+                    </clip>
+                    <noise>
+                        <type>gaussian</type>
+                        <mean>0.0</mean>
+                        <stddev>0.007</stddev>
+                    </noise>
+                </camera>
+                <plugin name="${base_name}_plugin" filename="libgazebo_ros_camera.so">
+                    <!-- <ros>
+                        <namespace>cam</namespace>
+                        <remapping>~/image_raw:=raw</remapping>
+                        <remapping>~/camera_info:=info</remapping>
+                    </ros> -->
+                    <!-- Set camera name. If empty, defaults to sensor name (i.e. "sensor_name") -->
+                    <camera_name>${base_name}</camera_name>
+                    <!-- Set TF frame name. If empty, defaults to link name (i.e. "link_name") -->
+                    <frame_name>${base_name}_optical_link</frame_name>
+                    <hack_baseline>0.2</hack_baseline>
+                </plugin>
+            </sensor>
+        </gazebo>
+    </xacro:macro>
 </robot>

File: robo_car_description/urdf/sensors/imu.xacro (robot description, xacro)
@@ -1,69 +1,68 @@
 <?xml version="1.0"?>
-<robot xmlns:xacro="http://www.ros.org/wiki/xacro"  name="robo_car">
-    <!-- <xacro:arg name="imu_visual"   default="true"/> -->
-  <!-- IMU LINK FRAME -->
-    <joint name="imu_joint" type="fixed">
-        <parent link="base_chassis_link"/>
-        <child link="imu_link"/>
-        <origin xyz="0 0 ${base_chassis_height}" rpy="0 0 0"/>
-        <axis xyz="0 0 0"/>
-    </joint>
-    <link name="imu_link"/>
-    <gazebo reference="imu_link">
-        <sensor name="imu" type="imu">
-            <always_on>true</always_on>
-            <update_rate>30</update_rate>
-            <visualize>$(arg imu_visual)</visualize>
-            <imu>
-            <angular_velocity>
-                <x>
-                <noise type="gaussian">
-                    <mean>0.0</mean>
-                    <stddev>2e-4</stddev>
-                </noise>
-                </x>
-                <y>
-                <noise type="gaussian">
-                    <mean>0.0</mean>
-                    <stddev>2e-4</stddev>
-                </noise>
-                </y>
-                <z>
-                <noise type="gaussian">
-                    <mean>0.0</mean>
-                    <stddev>2e-4</stddev>
-                </noise>
-                </z>
-            </angular_velocity>
-            <linear_acceleration>
-                <x>
-                <noise type="gaussian">
-                    <mean>0.0</mean>
-                    <stddev>1.7e-2</stddev>
-                </noise>
-                </x>
-                <y>
-                <noise type="gaussian">
-                    <mean>0.0</mean>
-                    <stddev>1.7e-2</stddev>
-                </noise>
-                </y>
-                <z>
-                <noise type="gaussian">
-                    <mean>0.0</mean>
-                    <stddev>1.7e-2</stddev>
-                </noise>
-                </z>
-            </linear_acceleration>
-            </imu>
-            <plugin name="imu_plugin" filename="libgazebo_ros_imu_sensor.so">
-                <ros>
-                    <namespace>imu</namespace>
-                    <remapping>~/out:=data</remapping>
-                </ros>
-                <initial_orientation_as_reference>false</initial_orientation_as_reference>
-                <frame_name>imu_link</frame_name>
-            </plugin>
-        </sensor>
-    </gazebo>
+<robot xmlns:xacro="http://www.ros.org/wiki/xacro">
+    <xacro:macro name="insert_imu" params="base_name parent_name x y z">
+        <joint name="${base_name}_joint" type="fixed">
+            <parent link="${parent_name}"/>
+            <child link="${base_name}"/>
+            <origin xyz="${x} ${y} ${z}" rpy="0 0 0"/>
+        </joint>
+        <link name="${base_name}"/>
+        <gazebo reference="${base_name}">
+            <sensor name="${base_name}" type="imu">
+                <always_on>true</always_on>
+                <update_rate>30</update_rate>
+                <visualize>true</visualize>
+                <imu>
+                    <angular_velocity>
+                        <x>
+                            <noise type="gaussian">
+                                <mean>0.0</mean>
+                                <stddev>2e-4</stddev>
+                            </noise>
+                        </x>
+                        <y>
+                            <noise type="gaussian">
+                                <mean>0.0</mean>
+                                <stddev>2e-4</stddev>
+                            </noise>
+                        </y>
+                        <z>
+                            <noise type="gaussian">
+                                <mean>0.0</mean>
+                                <stddev>2e-4</stddev>
+                            </noise>
+                        </z>
+                    </angular_velocity>
+                    <linear_acceleration>
+                        <x>
+                            <noise type="gaussian">
+                                <mean>0.0</mean>
+                                <stddev>1.7e-2</stddev>
+                            </noise>
+                        </x>
+                        <y>
+                            <noise type="gaussian">
+                                <mean>0.0</mean>
+                                <stddev>1.7e-2</stddev>
+                            </noise>
+                        </y>
+                        <z>
+                            <noise type="gaussian">
+                                <mean>0.0</mean>
+                                <stddev>1.7e-2</stddev>
+                            </noise>
+                        </z>
+                    </linear_acceleration>
+                </imu>
+                <plugin name="${base_name}_plugin" filename="libgazebo_ros_imu_sensor.so">
+                    <ros>
+                        <namespace>${base_name}</namespace>
+                        <remapping>~/out:=data</remapping>
+                    </ros>
+                    <initial_orientation_as_reference>false</initial_orientation_as_reference>
+                    <frame_name>${base_name}</frame_name>
+                </plugin>
+            </sensor>
+        </gazebo>
+    </xacro:macro>
 </robot>

File: robo_car_description/urdf/sensors/lidar.xacro (robot description, xacro)
@@ -1,66 +1,64 @@
 <?xml version="1.0"?>
-<robot xmlns:xacro="http://www.ros.org/wiki/xacro"  name="robo_car">
-    <!-- <xacro:arg name="laser_visual" default="false"/> -->
-    <!-- LIDAR LINK FRAME -->
-    <joint name="lidar_joint" type="fixed">
-        <parent link="base_chassis_link"/>
-        <child link="lidar_link"/>
-        <origin xyz="-0.05 0 ${full_chassis_height + 0.04}" rpy="0 0 0"/>
-        <axis xyz="0 0 0"/>
-    </joint>
-    <link name="lidar_link">
-    <visual>
-      <origin xyz="0 0 -0.02" rpy="0 0 0"/>
-      <geometry>
-        <cylinder radius="0.05" length="0.05" />
-      </geometry>
-      <material name="grey"/>
-    </visual>
-    <collision>
-      <origin xyz="0 0 -0.02" rpy="0 0 0"/>
-      <geometry>
-        <cylinder radius="0.05" length="0.05" />
-      </geometry>
-    </collision>
-    <xacro:inertial_cylinder mass="0.2" length="0.05" radius="0.05">
-            <origin xyz="0 0 -0.02" rpy="0 0 0"/>
-        </xacro:inertial_cylinder>
-    </link>
-    <gazebo reference="lidar_link">
-        <material>Gazebo/DarkGrey</material>
-        <sensor name="lidar" type="ray">
-            <always_on>true</always_on>
-            <visualize>$(arg laser_visual)</visualize>
-            <pose>0.0 0 0.0 0 0 0</pose>
-            <update_rate>15</update_rate>
-            <ray>
-                <scan>
-                <horizontal>
-                    <samples>720</samples>
-                    <resolution>1</resolution>
-                    <min_angle>${0*pi}</min_angle>
-                    <max_angle>${2*pi}</max_angle>
-                </horizontal>
-                </scan>
-                <range>
-                    <min>0.1</min>
-                    <max>5</max>
-                    <resolution>0.01</resolution>
-                </range>
-                <noise>
-                    <type>gaussian</type>
-                    <mean>0.0</mean>
-                    <stddev>0.01</stddev>
-                </noise>
-            </ray>
-            <plugin name="laser_plugin" filename="libgazebo_ros_ray_sensor.so">
-            <ros>
-                <namespace>lidar</namespace>
-                <remapping>~/out:=scan</remapping>
-            </ros>
-            <output_type>sensor_msgs/LaserScan</output_type>
-            <frame_name>lidar_link</frame_name>
-            </plugin>
-        </sensor>
-    </gazebo>
+<robot xmlns:xacro="http://www.ros.org/wiki/xacro" >
+    <xacro:macro name="insert_lidar" params="base_name parent_name x y z mass samples min_angle max_angle min_range max_range visualize">
+        <joint name="${base_name}_joint" type="fixed">
+            <parent link="${parent_name}"/>
+            <child link="${base_name}"/>
+            <origin xyz="${x} ${y} ${z}" rpy="0 0 0"/>
+        </joint>
+        <link name="${base_name}">
+            <visual>
+                <origin xyz="0 0 0"/>
+                <geometry>
+                    <cylinder radius="0.05" length="0.04"/>
+                </geometry>
+                <material name="black"/>
+            </visual>
+            <visual>
+                <origin xyz="0 0 -0.05"/>
+                <geometry>
+                    <cylinder radius="0.01" length="0.1"/>
+                </geometry>
+                <material name="black"/>
+            </visual>
+            <collision>
+                <geometry>
+                    <cylinder radius="0.05" length="0.04"/>
+                </geometry>
+            </collision>
+            <xacro:inertial_cylinder mass="${mass}" length="0.04" radius="0.05">
+                <origin xyz="0 0 0" rpy="0 0 0"/>
+            </xacro:inertial_cylinder>
+        </link>
+        <gazebo reference="${base_name}">
+            <material>Gazebo/DarkGrey</material>
+            <sensor name="${base_name}" type="ray">
+                <pose> 0 0 0 0 0 0 </pose>
+                <visualize>${visualize}</visualize>
+                <update_rate>10</update_rate>
+                <ray>
+                    <scan>
+                        <horizontal>
+                            <samples>${samples}</samples>
+                            <min_angle>${min_angle}</min_angle>
+                            <max_angle>${max_angle}</max_angle>
+                        </horizontal>
+                    </scan>
+                    <range>
+                        <min>${min_range}</min>
+                        <max>${max_range}</max>
+                    </range>
+                </ray>
+                <plugin name="${base_name}_plugin" filename="libgazebo_ros_ray_sensor.so">
+                    <ros>
+                        <namespace>${base_name}</namespace>
+                        <remapping>~/out:=scan</remapping>
+                        <!-- <argument>~/out:=scan</argument> -->
+                    </ros>
+                    <output_type>sensor_msgs/LaserScan</output_type>
+                    <frame_name>${base_name}</frame_name>
+                </plugin>
+            </sensor>
+        </gazebo>
+    </xacro:macro>
 </robot>
