Commit message: feat:updated robot description and drive controller

File: robo_car_description/urdf/sensors/sonar.xacro (robot description, xacro)
@@ -1,70 +1,70 @@
 <?xml version="1.0"?>
-<robot xmlns:xacro="http://www.ros.org/wiki/xacro"  name="robo_car">
+<robot xmlns:xacro="http://www.ros.org/wiki/xacro">
     <!-- <xacro:arg name="sonar_visual"   default="false"/> -->
-    <xacro:property name="deg2rad" value="0.017460317"/>
-    <xacro:property name="scan_angle" value="1"/>
-  <!-- SONAR LINK FRAME -->
-    <joint name="sonar_joint" type="fixed">
-        <parent link="base_chassis_link"/>
-        <child link="sonar_link"/>
-        <origin xyz="0.12 0 ${base_chassis_height/2}" rpy="0 0 0"/>
-        <axis xyz="0 0 0"/>
-    </joint>
-    <link name="sonar_link">
-        <visual>
-            <origin xyz="-0.015 0 0" rpy="0 ${pi/2} 0"/>
-            <geometry>
-                <cylinder radius="0.015" length="0.03" />
-            </geometry>
-            <material name="blue"/>
-        </visual>
-        <collision>
-            <origin xyz="-0.015 0 0" rpy="0 ${pi/2} 0"/>
-            <geometry>
-                <cylinder radius="0.0i5" length="0.03" />
-            </geometry>
-        </collision>
-        <xacro:inertial_cylinder mass="0.0005" length="0.03" radius="0.015">
-            <origin xyz="-0.015 0 0" rpy="0 0 0"/>
-        </xacro:inertial_cylinder>
-    </link>
-    <gazebo reference="sonar_link">
-        <material>Gazebo/Blue</material>
-        <sensor name="sonar" type="ray">
-            <always_on>true</always_on>
-            <visualize>$(arg sonar_visual)</visualize>
-            <pose>0.0 0 0.0 0 0 0</pose>
-            <update_rate>20</update_rate>
-            <ray>
-                <scan>
-                    <horizontal>
-                    <samples>20</samples>
-                    <resolution>1</resolution>
-                    <min_angle>${-scan_angle * deg2rad}</min_angle>
-                    <max_angle>${scan_angle * deg2rad}</max_angle>
-                    </horizontal>
-                    <vertical>
-                    <samples>20</samples>
-                    <resolution>1</resolution>
-                    <min_angle>${-scan_angle * deg2rad}</min_angle>
-                    <max_angle>${scan_angle * deg2rad}</max_angle>
-                    </vertical>
-                </scan>
-                <range>
-                    <min>0.01</min>
-                    <max>2</max>
-                    <resolution>0.02</resolution>
-                </range>
-            </ray>
-            <plugin name="sonar_plugin" filename="libgazebo_ros_ray_sensor.so">
-                <ros>
-                    <namespace>sonar</namespace>
-                    <remapping>~/out:=range</remapping>
-                </ros>
-                <output_type>sensor_msgs/Range</output_type>
-                <radiation_type>ultrasound</radiation_type>
-                <frame_name>sonar_link</frame_name>
-            </plugin>
-        </sensor>
-    </gazebo>
+    <!-- <xacro:property name="deg2rad" value="0.017460317"/>
+    <xacro:property name="scan_angle" value="1"/> -->
+    <xacro:macro name="insert_sonar" params="base_name parent_name x y z mass min_range max_range resolution visualize">
+        <joint name="${base_name}_joint" type="fixed">
+            <parent link="${parent_name}"/>
+            <child link="${base_name}"/>
+            <origin xyz="${x} ${y} ${z}" rpy="0 0 0"/>
+        </joint>
+        <link name="${base_name}">
+            <visual>
+                <origin xyz="-0.005 0 0" rpy="0 ${pi/2} 0"/>
+                <geometry>
+                    <cylinder radius="0.015" length="0.01" />
+                </geometry>
+                <material name="blue"/>
+            </visual>
+            <collision>
+                <origin xyz="-0.005 0 0" rpy="0 ${pi/2} 0"/>
+                <geometry>
+                    <cylinder radius="0.015" length="0.01" />
+                </geometry>
+            </collision>
+            <xacro:inertial_cylinder mass="${mass}" length="0.01" radius="0.01">
+                <origin xyz="-0.005 0 0" rpy="0 0 0"/>
+            </xacro:inertial_cylinder>
+        </link>
+        <gazebo reference="${base_name}">
+            <material>Gazebo/Blue</material>
+            <sensor name="${base_name}" type="ray">
+                <always_on>true</always_on>
+                <visualize>${visualize}</visualize>
+                <pose>0.0 0 0.0 0 0 0</pose>
+                <update_rate>5</update_rate>
+                <ray>
+                    <scan>
+                        <horizontal>
+                            <samples>20</samples>
+                            <resolution>1</resolution>
+                            <min_angle>${-pi/90}</min_angle>
+                            <max_angle>${pi/90}</max_angle>
+                        </horizontal>
+                        <vertical>
+                            <samples>20</samples>
+                            <resolution>1</resolution>
+                            <min_angle>${-pi/150}</min_angle>
+                            <max_angle>${pi/150}</max_angle>
+                        </vertical>
+                    </scan>
+                    <range>
+                        <min>${min_range}</min>
+                        <max>${max_range}</max>
+                        <resolution>${resolution}</resolution>
+                    </range>
+                </ray>
+                <plugin name="${base_name}_plugin" filename="libgazebo_ros_ray_sensor.so">
+                    <ros>
+                        <namespace>${base_name}</namespace>
+                        <remapping>~/out:=range</remapping>
+                    </ros>
+                    <output_type>sensor_msgs/Range</output_type>
+                    <radiation_type>ultrasound</radiation_type>
+                    <frame_name>${base_name}</frame_name>
+                </plugin>
+            </sensor>
+        </gazebo>
+    </xacro:macro>
 </robot>

File: robo_car_description/urdf/urdf_description.xacro (robot description, xacro)
@@ -5,4 +5,8 @@
     <xacro:include filename="$(find robo_car_description)/urdf/inertia_macros.xacro"/>
     <xacro:include filename="$(find robo_car_description)/urdf/face_macro.xacro"/>
+    <xacro:include filename="sensors/lidar.xacro"/>
+    <xacro:include filename="sensors/imu.xacro"/>
+    <xacro:include filename="sensors/cam.xacro"/>
+    <xacro:include filename="sensors/sonar.xacro"/>
     <xacro:property name="base_chassis_height" value="0.12"/>
     <xacro:property name="servo_mount_length" value="0.055"/>
@@ -25,5 +29,5 @@
     </joint>
     <link name="base_chassis_link">
-        <xacro:box_with_fillet size_x="0.4" size_y="0.30" size_z="${base_chassis_height}" fr="0.08" material="silver" x="0.15" y="0" z="${base_chassis_height/2}"/>
+        <xacro:box_with_fillet size_x="0.4" size_y="0.30" size_z="${base_chassis_height}" fr="0.08" material="white" x="0.15" y="0" z="${base_chassis_height/2}"/>
         <collision>
            <origin xyz="0.15 0 ${base_chassis_height/2}" rpy="0 0 0"/>
@@ -37,7 +41,7 @@
     </link>
     <gazebo reference="base_chassis_link">
-        <material>Gazebo/Silver</material>
-    </gazebo>
-    <xacro:insert_face parent_name="base_chassis_link" x="${0.15+0.2}" y="0" z="${base_chassis_height/2}"/>
+        <material>Gazebo/White</material>
+    </gazebo>
+    <!-- <xacro:insert_face parent_name="base_chassis_link" x="${0.15+0.2}" y="0" z="${base_chassis_height/2}"/> -->
     <!--  ########################### -->
     <!--  FRONT LEFT SERVO STEER LINK -->
@@ -450,7 +454,38 @@
     <!--  ########################### -->
     <xacro:include filename="$(find robo_car_description)/urdf/ros_controllers.xacro"/>
-    <!-- <xacro:include filename="$(find robo_car_description)/urdf/sensors/imu.xacro"/>
-    <xacro:include filename="$(find robo_car_description)/urdf/sensors/lidar.xacro"/>
-    <xacro:include filename="$(find robo_car_description)/urdf/sensors/cam.xacro"/>
-    <xacro:include filename="$(find robo_car_description)/urdf/sensors/sonar.xacro"/> -->
+       <!--  lidar -->
+    <xacro:property name="lidar_z_offset" value="0.1"/>
+    <xacro:insert_lidar
+        base_name="lidar"
+        parent_name="base_chassis_link"
+        x="0.15" y="0" z="${base_chassis_height+lidar_z_offset}"
+        mass="0.08" samples="360"
+        min_angle="${-pi*2}" max_angle="${pi*2}"
+        min_range="0.1" max_range="10"
+        visualize="false"/>
+    <!--  imu -->
+    <xacro:insert_imu
+        base_name="imu"
+        parent_name="base_chassis_link"
+        x="0" y="0" z="${base_chassis_height}"/>
+    <!--  normal camera style -->
+    <xacro:property name="cam_x_offset" value="0.04"/>
+    <xacro:property name="cam_z_offset" value="0.02"/>
+    <xacro:insert_camera
+        base_name="cam"
+        parent_name="base_chassis_link"
+        x="${0.15+0.2+cam_x_offset}" y="0" z="${base_chassis_height+cam_z_offset}"
+        mass="0.005"
+        width="640" height="480"
+        min_range="0.02" max_range="5.0"
+        tilt_angle="0"
+        visualize="true"/>
+    <!--  front sonar sensor -->
+    <xacro:insert_sonar
+        base_name="sonar"
+        parent_name="base_chassis_link"
+        x="${0.15+0.2+0.005}" y="0" z="${(base_chassis_height/2)}"
+        mass="0.0005"
+        min_range="0.02" max_range="3.0"
+        resolution="0.01" visualize="false"/>
 </robot>
