Commit message: sensor-setup-done

File: robo_car_description/urdf/part_macros.xacro (robot description, xacro)
@@ -130,58 +130,3 @@
         </xacro:inertial_cylinder>
     </xacro:macro>
-       <xacro:macro name="insert_rocker_link">
-        <visual>
-            <origin xyz="0 0 0" rpy="0 0 0"/>
-            <geometry>
-                <box size="${rocker_length} 0.05 0.02"/>
-            </geometry>
-            <material name="grey"/>
-        </visual>
-        <collision>
-            <origin xyz="0 0 0" rpy="0 0 0"/>
-            <geometry>
-                <box size="${rocker_length} 0.05 0.02"/>
-            </geometry>
-        </collision>
-        <xacro:inertial_box mass="0.2" x="${rocker_length}" y="0.05" z="0.02">
-            <origin xyz="0 0 0" rpy="0 0 0"/>
-        </xacro:inertial_box>
-    </xacro:macro>
-    <xacro:macro name="insert_boggie_link">
-        <visual>
-            <origin xyz="0 0 0" rpy="0 0 0"/>
-            <geometry>
-                <box size="0.05 ${boggie_length} 0.02"/>
-            </geometry>
-            <material name="grey"/>
-        </visual>
-        <collision>
-            <origin xyz="0 0 0" rpy="0 0 0"/>
-            <geometry>
-                <box size="0.05 ${boggie_length} 0.02"/>
-            </geometry>
-        </collision>
-        <xacro:inertial_box mass="0.2" x="0.05" y="${boggie_length}" z="0.2">
-            <origin xyz="0 0 0" rpy="0 0 0"/>
-        </xacro:inertial_box>
-    </xacro:macro>
-    <xacro:macro name="insert_servo_transmission" params="joint_name">
-        <joint name="${joint_name}">
-            <command_interface name="position">
-                <param name="min">${-pi/2}</param>
-                <param name="max">${pi/2}</param>
-            </command_interface>
-            <state_interface name="position"/>
-        </joint>
-    </xacro:macro>
-    <xacro:macro name="insert_wheel_transmission" params="joint_name">
-        <joint name="${joint_name}">
-            <command_interface name="velocity">
-                <param name="min">-10.0</param>
-                <param name="max">10.0</param>
-            </command_interface>
-            <state_interface name="position"/>
-            <state_interface name="velocity"/>
-        </joint>
-    </xacro:macro>
 </robot>

File: robo_car_description/urdf/ros_controllers.xacro (robot description, xacro)
@@ -29,6 +29,6 @@
             <joint_name>front_left_servo_joint</joint_name>
             <joint_name>front_right_servo_joint</joint_name>
-            <joint_name>rear_left_servo_joint</joint_name>
-            <joint_name>rear_right_servo_joint</joint_name>
+            <joint_name>front_left_wheel_joint</joint_name>
+            <joint_name>front_right_wheel_joint</joint_name>
             <joint_name>rear_left_wheel_joint</joint_name>
             <joint_name>rear_right_wheel_joint</joint_name>

File: robo_car_description/urdf/sensors/cam.xacro (robot description, xacro)
@@ -40,38 +40,25 @@
         <link name="${base_name}_optical_link"/>
         <gazebo reference="${base_name}">
-            <material>Gazebo/DarkGrey</material>
-            <sensor type="${base_name}" name="camera">
-                <visualize>${visualize}</visualize>
-                <update_rate>20.0</update_rate>
-                <camera name="${base_name}">
-                    <horizontal_fov>1.4</horizontal_fov>
-                    <image>
-                        <width>${width}</width>
-                        <height>${height}</height>
-                        <format>R8G8B8</format>
-                    </image>
-                    <clip>
-                        <near>${min_range}</near>
-                        <far>${max_range}</far>
-                    </clip>
-                    <noise>
-                        <type>gaussian</type>
-                        <mean>0.0</mean>
-                        <stddev>0.007</stddev>
-                    </noise>
-                </camera>
-                <plugin name="${base_name}_plugin" filename="libgazebo_ros_camera.so">
-                    <!-- <ros>
-                        <namespace>cam</namespace>
-                        <remapping>~/image_raw:=raw</remapping>
-                        <remapping>~/camera_info:=info</remapping>
-                    </ros> -->
-                    <!-- Set camera name. If empty, defaults to sensor name (i.e. "sensor_name") -->
-                    <camera_name>${base_name}</camera_name>
-                    <!-- Set TF frame name. If empty, defaults to link name (i.e. "link_name") -->
-                    <frame_name>${base_name}_optical_link</frame_name>
-                    <hack_baseline>0.2</hack_baseline>
-                </plugin>
-            </sensor>
+          <material>Gazebo/DarkGrey</material>
+          <sensor name="${base_name}" type="camera">
+            <pose> 0 0 0 0 0 0 </pose>
+            <visualize>${visualize}</visualize>
+            <update_rate>20</update_rate>
+            <camera>
+                <horizontal_fov>1.089</horizontal_fov>
+                <image>
+                    <format>R8G8B8</format>
+                    <width>${width}</width>
+                    <height>${height}</height>
+                </image>
+                <clip>
+                    <near>${min_range}</near>
+                    <far>${max_range}</far>
+                </clip>
+            </camera>
+            <plugin name="${base_name}_plugin" filename="libgazebo_ros_camera.so">
+                <frame_name>${base_name}_optical_link</frame_name>
+            </plugin>
+          </sensor>
         </gazebo>
     </xacro:macro>

File: robo_car_description/urdf/urdf_description.xacro (robot description, xacro)
@@ -5,16 +5,16 @@
     <xacro:include filename="$(find robo_car_description)/urdf/inertia_macros.xacro"/>
     <xacro:include filename="$(find robo_car_description)/urdf/face_macro.xacro"/>
-    <xacro:include filename="sensors/lidar.xacro"/>
-    <xacro:include filename="sensors/imu.xacro"/>
-    <xacro:include filename="sensors/cam.xacro"/>
-    <xacro:include filename="sensors/sonar.xacro"/>
+    <xacro:include filename="$(find robo_car_description)/urdf/sensors/lidar.xacro"/>
+    <xacro:include filename="$(find robo_car_description)/urdf/sensors/imu.xacro"/>
+    <xacro:include filename="$(find robo_car_description)/urdf/sensors/cam.xacro"/>
+    <xacro:include filename="$(find robo_car_description)/urdf/sensors/sonar.xacro"/>
     <xacro:property name="base_chassis_height" value="0.12"/>
     <xacro:property name="servo_mount_length" value="0.055"/>
     <xacro:property name="servo_mount_radius" value="0.01"/>
     <!-- <xacro:property name="support_radius" value="0.005"/> -->
-    <!-- <xacro:arg name="laser_visual" default="false"/>
+    <xacro:arg name="laser_visual" default="false"/>
     <xacro:arg name="imu_visual"   default="true"/>
     <xacro:arg name="sonar_visual"   default="false"/>
-    <xacro:arg name="cam_visual"   default="false"/> -->
+    <xacro:arg name="cam_visual"   default="false"/>
     <!-- BASE LINK -->
     <!-- <base joint/> -->
@@ -36,5 +36,5 @@
             </geometry>
         </collision>
-        <xacro:inertial_box mass="3" x="0.4" y="0.3" z="${base_chassis_height}">
+        <xacro:inertial_box mass="8.0" x="0.4" y="0.3" z="${base_chassis_height}">
             <origin xyz="0.15 0 ${base_chassis_height/2}" rpy="0 0 0"/>
         </xacro:inertial_box>
@@ -479,5 +479,5 @@
         width="640" height="480"
         min_range="0.02" max_range="5.0"
-        tilt_angle="0"
+        tilt_angle="${pi/72}"
         visualize="true"/>
     <!--  front sonar sensor -->
