Commit message: added race_track for self driving test

File: robo_car_description/urdf/drive_wheel_macro.xacro (robot description, xacro)
@@ -4,4 +4,9 @@
         <material name="black">
             <color rgba="0.1 0.1 0.1 1"/>
+        </material>
+    </xacro:macro>
+    <xacro:macro name="material_blue">
+        <material name="blue">
+            <color rgba="0.2 0.2 1 1"/>
         </material>
     </xacro:macro>
@@ -29,5 +34,5 @@
             <!-- <fdir1>1 0 0</fdir1> -->
             <minDepth>0.002</minDepth>
-            <material>Gazebo/FlatBlack</material>
+            <material>Gazebo/Blue</material>
         </gazebo>
     </xacro:macro>
@@ -51,5 +56,5 @@
                     <cylinder radius="${radius}" length="${thickness}"/>
                 </geometry>
-                <xacro:material_black/>
+                <xacro:material_blue/>
             </visual>
             <collision>

File: robo_car_description/urdf/sensors/cam.xacro (robot description, xacro)
@@ -46,5 +46,5 @@
             <update_rate>20</update_rate>
             <camera>
-                <horizontal_fov>1.089</horizontal_fov>
+                <horizontal_fov>1.46608</horizontal_fov>
                 <image>
                     <format>R8G8B8</format>

File: robo_car_description/urdf/urdf_description.xacro (robot description, xacro)
@@ -30,5 +30,5 @@
     </joint>
     <link name="chassis">
-        <xacro:box_with_fillet size_x="0.4" size_y="0.30" size_z="${chassis_height}" fr="0.08" material="white" x="0.15" y="0" z="${chassis_height/2}"/>
+        <xacro:box_with_fillet size_x="0.4" size_y="0.30" size_z="${chassis_height}" fr="0.08" material="orange" x="0.15" y="0" z="${chassis_height/2}"/>
         <collision>
            <origin xyz="0.15 0 ${chassis_height/2}" rpy="0 0 0"/>
@@ -42,5 +42,5 @@
     </link>
     <gazebo reference="chassis">
-        <material>Gazebo/White</material>
+        <material>Gazebo/Orange</material>
     </gazebo>
     <!-- <xacro:insert_face parent_name="chassis" x="${0.15+0.2}" y="0" z="${chassis_height/2}"/> -->
@@ -204,5 +204,5 @@
     <xacro:include filename="$(find robo_car_description)/urdf/ros_controllers.xacro"/>
        <!--  lidar -->
-    <xacro:property name="lidar_z_offset" value="0.1"/>
+    <!-- <xacro:property name="lidar_z_offset" value="0.1"/>
     <xacro:insert_lidar
         base_name="lidar"
@@ -212,5 +212,5 @@
         min_angle="${-pi*2}" max_angle="${pi*2}"
         min_range="0.1" max_range="10"
-        visualize="false"/>
+        visualize="false"/> -->
     <!--  imu -->
     <xacro:insert_imu
@@ -224,9 +224,9 @@
         base_name="cam"
         parent_name="chassis"
-        x="${0.15+0.2+cam_x_offset}" y="0" z="${chassis_height+cam_z_offset}"
+        x="${0.15+0.2+cam_x_offset-0.25}" y="0" z="${chassis_height+cam_z_offset+0.15}"
         mass="0.005"
         width="640" height="480"
         min_range="0.02" max_range="5.0"
-        tilt_angle="${pi/6}"
+        tilt_angle="${pi/16}"
         visualize="true"/>
     <!--  front sonar sensor -->

Commit message: feat added new design

File: robo_car_description/urdf/drive_wheel_macro.xacro (robot description, xacro)
@@ -1,4 +1,4 @@
 <?xml version="1.0"?>
-<robot name="mobo_bot" xmlns:xacro="http://www.ros.org/wiki/xacro" >
+<robot name="robo_car" xmlns:xacro="http://www.ros.org/wiki/xacro" >
     <xacro:macro name="material_black">
         <material name="black">
@@ -34,5 +34,5 @@
             <!-- <fdir1>1 0 0</fdir1> -->
             <minDepth>0.002</minDepth>
-            <material>Gazebo/Blue</material>
+            <material>Gazebo/FlatBlack</material>
         </gazebo>
     </xacro:macro>
@@ -56,5 +56,5 @@
                     <cylinder radius="${radius}" length="${thickness}"/>
                 </geometry>
-                <xacro:material_blue/>
+                <xacro:material_black/>
             </visual>
             <collision>

File: robo_car_description/urdf/sensors/lidar.xacro (robot description, xacro)
@@ -13,5 +13,5 @@
                     <cylinder radius="0.05" length="0.04"/>
                 </geometry>
-                <material name="black"/>
+                <material name="grey"/>
             </visual>
             <visual>
@@ -20,5 +20,5 @@
                     <cylinder radius="0.01" length="0.1"/>
                 </geometry>
-                <material name="black"/>
+                <material name="grey"/>
             </visual>
             <collision>

File: robo_car_description/urdf/urdf_description.xacro (robot description, xacro)
@@ -5,5 +5,5 @@
     <xacro:include filename="$(find robo_car_description)/urdf/inertia_macros.xacro"/>
     <xacro:include filename="$(find robo_car_description)/urdf/drive_wheel_macro.xacro"/>
-    <xacro:include filename="$(find robo_car_description)/urdf/face_macro.xacro"/>
+    <xacro:include filename="$(find robo_car_description)/urdf/ros_controllers.xacro"/>
     <xacro:include filename="$(find robo_car_description)/urdf/sensors/lidar.xacro"/>
     <xacro:include filename="$(find robo_car_description)/urdf/sensors/imu.xacro"/>
@@ -14,8 +14,7 @@
     <xacro:property name="wheel_mass" value="0.04"/>
     <xacro:property name="spoke_width" value="0.01"/>
-    <xacro:property name="chassis_height" value="0.12"/>
-    <xacro:property name="servo_mount_length" value="0.055"/>
-    <xacro:property name="servo_mount_radius" value="0.01"/>
-    <!-- <xacro:property name="support_radius" value="0.005"/> -->
+    <xacro:property name="chassis_height" value="0.075"/>
+    <xacro:property name="wheel_seperation" value="0.26"/>
+    <xacro:property name="dist_btw_front_rear" value="0.3"/>
     <!-- BASE LINK -->
     <!-- <base joint/> -->
@@ -27,15 +26,46 @@
         <parent link="base_link"/>
         <child link="chassis"/>
-        <origin xyz="0 0 0.101"/>
+        <origin xyz="0 0 0.05"/>
     </joint>
     <link name="chassis">
-        <xacro:box_with_fillet size_x="0.4" size_y="0.30" size_z="${chassis_height}" fr="0.08" material="orange" x="0.15" y="0" z="${chassis_height/2}"/>
+        <xacro:box_with_fillet size_x="0.28" size_y="0.2" size_z="${chassis_height}" fr="0.02" material="orange" x="0.09" y="0" z="${chassis_height/2}"/>
+        <collision>
+           <origin xyz="0.09 0 ${chassis_height/2}" rpy="0 0 0"/>
+            <geometry>
+                <box size="0.28 0.2 ${chassis_height}"/>
+            </geometry>
+        </collision>
+        <xacro:box_with_fillet size_x="0.4" size_y="0.1" size_z="${chassis_height}" fr="0.02" material="orange" x="0.15" y="0" z="${chassis_height/2}"/>
         <collision>
            <origin xyz="0.15 0 ${chassis_height/2}" rpy="0 0 0"/>
             <geometry>
-                <box size="0.4 0.3 ${chassis_height}"/>
-            </geometry>
-        </collision>
-        <xacro:inertial_box mass="2.0" x="0.4" y="0.3" z="${chassis_height}">
+                <box size="0.4 0.1 ${chassis_height}"/>
+            </geometry>
+        </collision>
+        <visual>
+            <origin xyz="0 0 0" rpy="${-pi/2} 0 0"/>
+            <geometry>
+                <cylinder length="${wheel_seperation-0.04}" radius="0.01"/>
+            </geometry>
+        </visual>
+        <collision>
+           <origin xyz="0 0 0" rpy="${-pi/2} 0 0"/>
+            <geometry>
+                <cylinder length="${wheel_seperation-0.04}" radius="0.01"/>
+            </geometry>
+        </collision>
+        <visual>
+            <origin xyz="${dist_btw_front_rear} 0 0" rpy="${-pi/2} 0 0"/>
+            <geometry>
+                <cylinder length="${wheel_seperation-0.04}" radius="0.01"/>
+            </geometry>
+        </visual>
+        <collision>
+           <origin xyz="${dist_btw_front_rear} 0 0" rpy="${-pi/2} 0 0"/>
+            <geometry>
+                <cylinder length="${wheel_seperation-0.04}" radius="0.01"/>
+            </geometry>
+        </collision>
+        <xacro:inertial_box mass="4.0" x="0.4" y="0.2" z="${chassis_height}">
             <origin xyz="0.15 0 ${chassis_height/2}" rpy="0 0 0"/>
         </xacro:inertial_box>
@@ -44,5 +74,4 @@
         <material>Gazebo/Orange</material>
     </gazebo>
-    <!-- <xacro:insert_face parent_name="chassis" x="${0.15+0.2}" y="0" z="${chassis_height/2}"/> -->
     <!--  ########################### -->
     <!--  FRONT LEFT SERVO STEER LINK -->
@@ -50,5 +79,5 @@
         <parent link="chassis"/>
         <child link="front_left_servo"/>
-        <origin xyz="0.3 ${0.15-servo_mount_radius} 0"/>
+        <origin xyz="${dist_btw_front_rear} 0.1 0"/>
         <axis xyz="0 0 1"/>
         <limit effort="1000.0" lower="${-pi/2}" upper="${pi/2}" velocity="0.5"/>
@@ -56,18 +85,18 @@
     <link name="front_left_servo">
         <visual>
-            <origin xyz="0 0 ${-servo_mount_length/2}" rpy="0 0 0"/>
-            <geometry>
-                <cylinder radius="${servo_mount_radius}" length="${servo_mount_length}"/>
+            <origin xyz="0 0 0" rpy="0 0 0"/>
+            <geometry>
+                <cylinder radius="0.01" length="0.02"/>
             </geometry>
             <material name="black"/>
         </visual>
         <collision>
-           <origin xyz="0 0 ${-servo_mount_length/2}" rpy="0 0 0"/>
-            <geometry>
-                <cylinder radius="${servo_mount_radius}" length="${servo_mount_length}"/>
-            </geometry>
-        </collision>
-        <xacro:inertial_cylinder mass="0.005" length="${servo_mount_length}" radius="${servo_mount_radius}">
-            <origin xyz="0 0 ${-servo_mount_length/2}" rpy="0 0 0"/>
+           <origin xyz="0 0 0" rpy="0 0 0"/>
+            <geometry>
+                <cylinder radius="0.01" length="0.02"/>
+            </geometry>
+        </collision>
+        <xacro:inertial_cylinder mass="0.005" length="0.02" radius="0.01">
+            <origin xyz="0 0 0" rpy="0 0 0"/>
         </xacro:inertial_cylinder>
     </link>
@@ -75,20 +104,20 @@
         <material>Gazebo/DarkGrey</material>
     </gazebo>
-    <!--  ########################### -->
-    <!--  FRONT LEFT WHEEL LINK -->
+    <!-- ############################### -->
+    <!-- FRONT LEFT DRIVE WHEELS -->
     <xacro:insert_drive_wheel
         base_name="front_left_wheel"
         parent_name="front_left_servo"
-        x="0" y="${servo_mount_radius+0.021}" z="-0.051"
-        mass="${wheel_mass}"
-        radius="${wheel_radius}"
-        thickness="${wheel_width}"
-        spoke_width="${spoke_width}"/>
-    <!--  ########################### -->
+        x="0" y="0.03" z="0"
+        mass="${wheel_mass}"
+        radius="${wheel_radius}"
+        thickness="${wheel_width}"
+        spoke_width="${spoke_width}"/>
+    <!-- ############################### -->
     <!--  FRONT RIGHT SERVO STEER LINK -->
     <joint name="front_right_servo_joint" type="revolute">
         <parent link="chassis"/>
         <child link="front_right_servo"/>
-        <origin xyz="0.3 ${-0.15+servo_mount_radius} 0"/>
+        <origin xyz="${dist_btw_front_rear} -0.1 0"/>
         <axis xyz="0 0 1"/>
         <limit effort="1000.0" lower="${-pi/2}" upper="${pi/2}" velocity="0.5"/>
@@ -96,18 +125,18 @@
     <link name="front_right_servo">
         <visual>
-            <origin xyz="0 0 ${-servo_mount_length/2}" rpy="0 0 0"/>
-            <geometry>
-                <cylinder radius="${servo_mount_radius}" length="${servo_mount_length}"/>
+            <origin xyz="0 0 0" rpy="0 0 0"/>
+            <geometry>
+                <cylinder radius="0.01" length="0.02"/>
             </geometry>
             <material name="black"/>
         </visual>
         <collision>
-           <origin xyz="0 0 ${-servo_mount_length/2}" rpy="0 0 0"/>
-            <geometry>
-                <cylinder radius="${servo_mount_radius}" length="${servo_mount_length}"/>
-            </geometry>
-        </collision>
-        <xacro:inertial_cylinder mass="0.005" length="${servo_mount_length}" radius="${servo_mount_radius}">
-            <origin xyz="0 0 ${-servo_mount_length/2}" rpy="0 0 0"/>
+           <origin xyz="0 0 0" rpy="0 0 0"/>
+            <geometry>
+                <cylinder radius="0.01" length="0.02"/>
+            </geometry>
+        </collision>
+        <xacro:inertial_cylinder mass="0.005" length="0.02" radius="0.01">
+            <origin xyz="0 0 0" rpy="0 0 0"/>
         </xacro:inertial_cylinder>
     </link>
@@ -115,94 +144,35 @@
         <material>Gazebo/DarkGrey</material>
     </gazebo>
-    <!--  ########################### -->
-    <!--  FRONT RIGHT WHEEL LINK -->
+    <!-- ############################### -->
+    <!-- FRONT RIGHT DRIVE WHEEL -->
     <xacro:insert_drive_wheel
         base_name="front_right_wheel"
         parent_name="front_right_servo"
-        x="0" y="${-1*(servo_mount_radius+0.021)}" z="-0.051"
-        mass="${wheel_mass}"
-        radius="${wheel_radius}"
-        thickness="${wheel_width}"
-        spoke_width="${spoke_width}"/>
-    <!--  ########################### -->
-    <!--  REAR LEFT SERVO STEER LINK -->
-    <joint name="rear_left_servo_joint" type="fixed">
-        <parent link="chassis"/>
-        <child link="rear_left_servo"/>
-        <origin xyz="0 ${0.15-servo_mount_radius} 0"/>
-    </joint>
-    <link name="rear_left_servo">
-        <visual>
-            <origin xyz="0 0 ${-servo_mount_length/2}" rpy="0 0 0"/>
-            <geometry>
-                <cylinder radius="${servo_mount_radius}" length="${servo_mount_length}"/>
-            </geometry>
-            <material name="black"/>
-        </visual>
-        <collision>
-           <origin xyz="0 0 ${-servo_mount_length/2}" rpy="0 0 0"/>
-            <geometry>
-                <cylinder radius="${servo_mount_radius}" length="${servo_mount_length}"/>
-            </geometry>
-        </collision>
-        <xacro:inertial_cylinder mass="0.005" length="${servo_mount_length}" radius="${servo_mount_radius}">
-            <origin xyz="0 0 ${-servo_mount_length/2}" rpy="0 0 0"/>
-        </xacro:inertial_cylinder>
-    </link>
-    <gazebo reference="rear_left_servo">
-        <material>Gazebo/DarkGrey</material>
-    </gazebo>
-    <!--  ########################### -->
-    <!--  REAR LEFT WHEEL LINK -->
+        x="0" y="-0.03" z="0"
+        mass="${wheel_mass}"
+        radius="${wheel_radius}"
+        thickness="${wheel_width}"
+        spoke_width="${spoke_width}"/>
+    <!-- ############################### -->
+    <!-- REAR LEFT AND RIGHT DRIVE WHEELS -->
     <xacro:insert_drive_wheel
         base_name="rear_left_wheel"
-        parent_name="rear_left_servo"
-        x="0" y="${servo_mount_radius+0.021}" z="-0.051"
-        mass="${wheel_mass}"
-        radius="${wheel_radius}"
-        thickness="${wheel_width}"
-        spoke_width="${spoke_width}"/>
-    <!--  ########################### -->
-    <!--  FRONT RIGHT SERVO STEER LINK -->
-    <joint name="rear_right_servo_joint" type="fixed">
-        <parent link="chassis"/>
-        <child link="rear_right_servo"/>
-        <origin xyz="0 ${-0.15+servo_mount_radius} 0"/>
-    </joint>
-    <link name="rear_right_servo">
-        <visual>
-            <origin xyz="0 0 ${-servo_mount_length/2}" rpy="0 0 0"/>
-            <geometry>
-                <cylinder radius="${servo_mount_radius}" length="${servo_mount_length}"/>
-            </geometry>
-            <material name="black"/>
-        </visual>
-        <collision>
-           <origin xyz="0 0 ${-servo_mount_length/2}" rpy="0 0 0"/>
-            <geometry>
-                <cylinder radius="${servo_mount_radius}" length="${servo_mount_length}"/>
-            </geometry>
-        </collision>
-        <xacro:inertial_cylinder mass="0.005" length="${servo_mount_length}" radius="${servo_mount_radius}">
-            <origin xyz="0 0 ${-servo_mount_length/2}" rpy="0 0 0"/>
-        </xacro:inertial_cylinder>
-    </link>
-    <gazebo reference="rear_right_servo">
-        <material>Gazebo/DarkGrey</material>
-    </gazebo>
-    <!--  ########################### -->
-    <!--  REAR RIGHT WHEEL LINK -->
+        parent_name="chassis"
+        x="0" y="${wheel_seperation/2}" z="0"
+        mass="${wheel_mass}"
+        radius="${wheel_radius}"
+        thickness="${wheel_width}"
+        spoke_width="${spoke_width}"/>
     <xacro:insert_drive_wheel
         base_name="rear_right_wheel"
-        parent_name="rear_right_servo"
-        x="0" y="${-1*(servo_mount_radius+0.021)}" z="-0.051"
-        mass="${wheel_mass}"
-        radius="${wheel_radius}"
-        thickness="${wheel_width}"
-        spoke_width="${spoke_width}"/>
-    <!--  ########################### -->
-    <xacro:include filename="$(find robo_car_description)/urdf/ros_controllers.xacro"/>
-       <!--  lidar -->
-    <!-- <xacro:property name="lidar_z_offset" value="0.1"/>
+        parent_name="chassis"
+        x="0" y="${-wheel_seperation/2}" z="0"
+        mass="${wheel_mass}"
+        radius="${wheel_radius}"
+        thickness="${wheel_width}"
+        spoke_width="${spoke_width}"/>
+    <!-- ############################### -->
+    <!--  lidar -->
+    <xacro:property name="lidar_z_offset" value="0.1"/>
     <xacro:insert_lidar
         base_name="lidar"
@@ -212,5 +182,5 @@
         min_angle="${-pi*2}" max_angle="${pi*2}"
         min_range="0.1" max_range="10"
-        visualize="false"/> -->
+        visualize="false"/>
     <!--  imu -->
     <xacro:insert_imu
@@ -224,10 +194,49 @@
         base_name="cam"
         parent_name="chassis"
-        x="${0.15+0.2+cam_x_offset-0.25}" y="0" z="${chassis_height+cam_z_offset+0.15}"
+        x="0.15" y="0" z="${chassis_height+cam_z_offset+0.15}"
         mass="0.005"
         width="640" height="480"
         min_range="0.02" max_range="5.0"
-        tilt_angle="${pi/16}"
-        visualize="true"/>
+        tilt_angle="${pi/20}"
+        visualize="false"/>
+    <joint name="cam_stand_joint" type="fixed">
+        <parent link="chassis"/>
+        <child link="cam_stand"/>
+        <origin xyz="0.05 0 0"/>
+    </joint>
+    <link name="cam_stand">
+        <visual>
+            <origin xyz="0 0 ${(chassis_height+cam_z_offset+0.15)/2}" rpy="0 0 0"/>
+            <geometry>
+                <cylinder radius="0.01" length="${chassis_height+cam_z_offset+0.15}"/>
+            </geometry>
+            <material name="white"/>
+        </visual>
+        <collision>
+           <origin xyz="0 0 ${(chassis_height+cam_z_offset+0.15)/2}" rpy="0 0 0"/>
+            <geometry>
+                <cylinder radius="0.01" length="${chassis_height+cam_z_offset+0.15}"/>
+            </geometry>
+        </collision>
+        <visual>
+            <origin xyz="${(0.08/2)-0.01} 0 ${chassis_height+cam_z_offset+0.15}" rpy="0 ${-pi/2} 0"/>
+            <geometry>
+                <cylinder radius="0.01" length="0.08"/>
+            </geometry>
+            <material name="white"/>
+        </visual>
+        <collision>
+           <origin xyz="${(0.08/2)-0.01} 0 ${chassis_height+cam_z_offset+0.15}" rpy="0 ${-pi/2} 0"/>
+            <geometry>
+                <cylinder radius="0.01" length="0.08"/>
+            </geometry>
+        </collision>
+        <xacro:inertial_cylinder mass="0.005" length="0.02" radius="0.01">
+            <origin xyz="0 0 0" rpy="0 0 0"/>
+        </xacro:inertial_cylinder>
+    </link>
+    <gazebo reference="cam_stand">
+        <material>Gazebo/White</material>
+    </gazebo>
     <!--  front sonar sensor -->
     <xacro:insert_sonar
