Commit message: updated robot design

File: robo_car_description/urdf/color_macros.xacro (robot description, xacro)
@@ -1,4 +1,4 @@
 <?xml version="1.0"?>
-<robot name="robo_car" xmlns:xacro="http://www.ros.org/wiki/xacro" >
+<robot xmlns:xacro="http://www.ros.org/wiki/xacro" >
     <material name="white">
         <color rgba="1 1 1 1" />

File: robo_car_description/urdf/controllers/gazebo_hw_ros2_control.xacro (robot description, xacro)
@@ -1,5 +1,5 @@
 <?xml version="1.0"?>
-<robot name="robo_car" xmlns:xacro="http://ros.org/wiki/xacro">
-    <xacro:include filename="$(find robo_car_description)/urdf/transmission_macros.xacro"/>
+<robot xmlns:xacro="http://ros.org/wiki/xacro">
+    <xacro:include filename="transmission_macros.xacro"/>
     <ros2_control name="GazeboSystem" type="system">
         <hardware>

File: robo_car_description/urdf/controllers/transmission_macros.xacro (robot description, xacro)
@@ -1,4 +1,4 @@
 <?xml version="1.0"?>
-<robot xmlns:xacro="http://www.ros.org/wiki/xacro" name="robo_car">
+<robot xmlns:xacro="http://www.ros.org/wiki/xacro">
     <xacro:macro name="insert_servo_transmission" params="joint_name">
         <joint name="${joint_name}">

File: robo_car_description/urdf/robot_core.xacro (robot description, xacro)
@@ -1,17 +1,15 @@
 <?xml version="1.0"?>
-<robot xmlns:xacro="http://www.ros.org/wiki/xacro"  name="robo_car">
-    <xacro:include filename="$(find robo_car_description)/urdf/color_materials.xacro"/>
-    <xacro:include filename="$(find robo_car_description)/urdf/part_macros.xacro"/>
-    <xacro:include filename="$(find robo_car_description)/urdf/inertia_macros.xacro"/>
-    <xacro:include filename="$(find robo_car_description)/urdf/drive_wheel_macro.xacro"/>
-    <xacro:include filename="$(find robo_car_description)/urdf/ros_controllers.xacro"/>
-    <xacro:include filename="$(find robo_car_description)/urdf/sensors/lidar.xacro"/>
-    <xacro:include filename="$(find robo_car_description)/urdf/sensors/imu.xacro"/>
-    <xacro:include filename="$(find robo_car_description)/urdf/sensors/cam.xacro"/>
-    <xacro:include filename="$(find robo_car_description)/urdf/sensors/sonar.xacro"/>
+<robot xmlns:xacro="http://www.ros.org/wiki/xacro">
+    <xacro:include filename="other_parts/box_with_fillet_macro.xacro"/>
+    <xacro:include filename="other_parts/drive_wheel_macro.xacro"/>
+    <xacro:include filename="other_parts/drive_wheel_rim_macro.xacro"/>
+    <xacro:include filename="sensors/sonar.xacro"/>
+    <xacro:include filename="sensors/lidar.xacro"/>
+    <!-- <xacro:include filename="sensors/imu.xacro"/> -->
+    <xacro:include filename="sensors/cam.xacro"/>
     <xacro:property name="wheel_radius" value="0.05"/>
     <xacro:property name="wheel_width" value="0.04"/>
     <xacro:property name="wheel_mass" value="0.04"/>
-    <xacro:property name="spoke_width" value="0.01"/>
+    <xacro:property name="spoke_width" value="0.0075"/>
     <xacro:property name="chassis_height" value="0.075"/>
     <xacro:property name="wheel_seperation" value="0.26"/>
@@ -29,5 +27,6 @@
     </joint>
     <link name="chassis">
-        <xacro:box_with_fillet size_x="0.28" size_y="0.2" size_z="${chassis_height}" fr="0.02" material="orange" x="0.09" y="0" z="${chassis_height/2}"/>
+        <xacro:insert_box_with_fillet size_x="0.28" size_y="0.2" size_z="${chassis_height}"
+        fillet_radius="0.02" material="orange" x="0.09" y="0" z="${chassis_height/2}"/>
         <collision>
            <origin xyz="0.09 0 ${chassis_height/2}" rpy="0 0 0"/>
@@ -36,5 +35,6 @@
             </geometry>
         </collision>
-        <xacro:box_with_fillet size_x="0.4" size_y="0.1" size_z="${chassis_height}" fr="0.02" material="orange" x="0.15" y="0" z="${chassis_height/2}"/>
+        <xacro:insert_box_with_fillet size_x="0.4" size_y="0.1" size_z="${chassis_height}"
+        fillet_radius="0.02" material="orange" x="0.15" y="0" z="${chassis_height/2}"/>
         <collision>
            <origin xyz="0.15 0 ${chassis_height/2}" rpy="0 0 0"/>
@@ -105,5 +105,5 @@
     </gazebo>
     <!-- ############################### -->
-    <!-- FRONT LEFT DRIVE WHEELS -->
+    <!-- FRONT LEFT DRIVE WHEEL -->
     <xacro:insert_drive_wheel
         base_name="front_left_wheel"
@@ -112,7 +112,13 @@
         mass="${wheel_mass}"
         radius="${wheel_radius}"
-        thickness="${wheel_width}"
-        spoke_width="${spoke_width}"/>
-    <!-- ############################### -->
+        thickness="${wheel_width}"/>
+    <xacro:insert_drive_wheel_rim
+        base_name="front_left_rim"
+        parent_name="front_left_wheel"
+        x="0" y="0" z="0.001"
+        radius="${wheel_radius}"
+        thickness="${wheel_width}"
+        spoke_width="${spoke_width}"/>
+    <!-- ############################# -->
     <!--  FRONT RIGHT SERVO STEER LINK -->
     <joint name="front_right_servo_joint" type="revolute">
@@ -152,8 +158,14 @@
         mass="${wheel_mass}"
         radius="${wheel_radius}"
-        thickness="${wheel_width}"
-        spoke_width="${spoke_width}"/>
-    <!-- ############################### -->
-    <!-- REAR LEFT AND RIGHT DRIVE WHEELS -->
+        thickness="${wheel_width}"/>
+    <xacro:insert_drive_wheel_rim
+        base_name="front_right_rim"
+        parent_name="front_right_wheel"
+        x="0" y="0" z="-0.001"
+        radius="${wheel_radius}"
+        thickness="${wheel_width}"
+        spoke_width="${spoke_width}"/>
+    <!-- ############################### -->
+    <!-- REAR LEFT DRIVE WHEEL -->
     <xacro:insert_drive_wheel
         base_name="rear_left_wheel"
@@ -162,6 +174,14 @@
         mass="${wheel_mass}"
         radius="${wheel_radius}"
-        thickness="${wheel_width}"
-        spoke_width="${spoke_width}"/>
+        thickness="${wheel_width}"/>
+    <xacro:insert_drive_wheel_rim
+        base_name="rear_left_rim"
+        parent_name="rear_left_wheel"
+        x="0" y="0" z="0.001"
+        radius="${wheel_radius}"
+        thickness="${wheel_width}"
+        spoke_width="${spoke_width}"/>
+    <!-- ############################### -->
+    <!-- REAR RIGHT DRIVE WHEEL -->
     <xacro:insert_drive_wheel
         base_name="rear_right_wheel"
@@ -170,22 +190,36 @@
         mass="${wheel_mass}"
         radius="${wheel_radius}"
-        thickness="${wheel_width}"
-        spoke_width="${spoke_width}"/>
-    <!-- ############################### -->
-    <!--  lidar -->
-    <xacro:property name="lidar_z_offset" value="0.1"/>
+        thickness="${wheel_width}"/>
+    <xacro:insert_drive_wheel_rim
+        base_name="rear_right_rim"
+        parent_name="rear_right_wheel"
+        x="0" y="0" z="-0.001"
+        radius="${wheel_radius}"
+        thickness="${wheel_width}"
+        spoke_width="${spoke_width}"/>
+    <!-- ############################# -->
+    <!--  sonar -->
+    <xacro:insert_sonar
+        base_name="sonar"
+        parent_name="chassis"
+        x="${0.15+0.2+0.005}" y="0" z="${(chassis_height/2)}"
+        mass="0.005"
+        min_range="0.02" max_range="3.0"
+        resolution="0.01" visualize="false"/>
+     <!--  lidar -->
+    <xacro:property name="lidar_z_offset" value="0.04"/>
     <xacro:insert_lidar
         base_name="lidar"
         parent_name="chassis"
-        x="0.15" y="0" z="${chassis_height+lidar_z_offset}"
-        mass="0.08" samples="360"
+        x="0.2" y="0" z="${chassis_height+lidar_z_offset}"
+        mass="0.1" samples="360"
         min_angle="${-pi*2}" max_angle="${pi*2}"
         min_range="0.1" max_range="10"
         visualize="false"/>
     <!--  imu -->
-    <xacro:insert_imu
+    <!-- <xacro:insert_imu
         base_name="imu"
         parent_name="chassis"
-        x="0" y="0" z="${chassis_height}"/>
+        x="0" y="0" z="${chassis_height}"/> -->
     <!--  normal camera style -->
     <xacro:property name="cam_x_offset" value="0.04"/>
@@ -199,51 +233,4 @@
         min_range="0.02" max_range="5.0"
         tilt_angle="${pi/20}"
-        visualize="false"/>
-    <joint name="cam_stand_joint" type="fixed">
-        <parent link="chassis"/>
-        <child link="cam_stand"/>
-        <origin xyz="0.05 0 0"/>
-    </joint>
-    <link name="cam_stand">
-        <visual>
-            <origin xyz="0 0 ${(chassis_height+cam_z_offset+0.15)/2}" rpy="0 0 0"/>
-            <geometry>
-                <cylinder radius="0.01" length="${chassis_height+cam_z_offset+0.15}"/>
-            </geometry>
-            <material name="white"/>
-        </visual>
-        <collision>
-           <origin xyz="0 0 ${(chassis_height+cam_z_offset+0.15)/2}" rpy="0 0 0"/>
-            <geometry>
-                <cylinder radius="0.01" length="${chassis_height+cam_z_offset+0.15}"/>
-            </geometry>
-        </collision>
-        <visual>
-            <origin xyz="${(0.08/2)-0.01} 0 ${chassis_height+cam_z_offset+0.15}" rpy="0 ${-pi/2} 0"/>
-            <geometry>
-                <cylinder radius="0.01" length="0.08"/>
-            </geometry>
-            <material name="white"/>
-        </visual>
-        <collision>
-           <origin xyz="${(0.08/2)-0.01} 0 ${chassis_height+cam_z_offset+0.15}" rpy="0 ${-pi/2} 0"/>
-            <geometry>
-                <cylinder radius="0.01" length="0.08"/>
-            </geometry>
-        </collision>
-        <xacro:inertial_cylinder mass="0.005" length="0.02" radius="0.01">
-            <origin xyz="0 0 0" rpy="0 0 0"/>
-        </xacro:inertial_cylinder>
-    </link>
-    <gazebo reference="cam_stand">
-        <material>Gazebo/White</material>
-    </gazebo>
-    <!--  front sonar sensor -->
-    <xacro:insert_sonar
-        base_name="sonar"
-        parent_name="chassis"
-        x="${0.15+0.2+0.005}" y="0" z="${(chassis_height/2)}"
-        mass="0.0005"
-        min_range="0.02" max_range="3.0"
-        resolution="0.01" visualize="false"/>
+        visualize="true"/>
 </robot>

File: robo_car_description/urdf/sensors/cam.xacro (robot description, xacro)
@@ -46,4 +46,5 @@
             <update_rate>20</update_rate>
             <camera>
+                <!-- <horizontal_fov>1.089</horizontal_fov> -->
                 <horizontal_fov>1.46608</horizontal_fov>
                 <image>
@@ -64,2 +65,44 @@
     </xacro:macro>
 </robot>
+ <!-- <joint name="line_cam_joint" type="fixed">
+        <parent link="chassis"/>
+        <child link="line_cam"/>
+        <origin xyz="0.305 0 0.08" rpy="0 0 0"/>
+    </joint>
+    <link name="line_cam">
+        <visual>
+            <geometry>
+                <box size="0.010 0.03 0.03"/>
+            </geometry>
+            <material name="red"/>
+        </visual>
+    </link>
+    <joint name="line_cam_optical_joint" type="fixed">
+        <parent link="line_cam"/>
+        <child link="line_cam_link_optical"/>
+        <origin xyz="0 0 0" rpy="${-pi/2} 0 ${-pi/2}"/>
+    </joint>
+    <link name="line_cam_link_optical"></link>
+    <gazebo reference="line_cam">
+        <material>Gazebo/Red</material>
+        <sensor name="line_cam" type="camera">
+            <pose> 0 0 0 0 0 0 </pose>
+            <visualize>true</visualize>
+            <update_rate>10</update_rate>
+            <camera>
+                <horizontal_fov>1.089</horizontal_fov>
+                <image>
+                    <format>R8G8B8</format>
+                    <width>640</width>
+                    <height>480</height>
+                </image>
+                <clip>
+                    <near>0.05</near>
+                    <far>8.0</far>
+                </clip>
+            </camera>
+            <plugin name="camera_controller" filename="libgazebo_ros_camera.so">
+                <frame_name>line_cam_link_optical</frame_name>
+            </plugin>
+        </sensor>
+    </gazebo> -->

File: robo_car_description/urdf/sensors/lidar.xacro (robot description, xacro)
@@ -9,24 +9,18 @@
         <link name="${base_name}">
             <visual>
-                <origin xyz="0 0 0"/>
+                <origin xyz="0 0 -0.02"/>
                 <geometry>
-                    <cylinder radius="0.05" length="0.04"/>
-                </geometry>
-                <material name="grey"/>
-            </visual>
-            <visual>
-                <origin xyz="0 0 -0.05"/>
-                <geometry>
-                    <cylinder radius="0.01" length="0.1"/>
+                    <cylinder radius="0.03" length="0.04"/>
                 </geometry>
                 <material name="grey"/>
             </visual>
             <collision>
+                <origin xyz="0 0 -0.02"/>
                 <geometry>
-                    <cylinder radius="0.05" length="0.04"/>
+                    <cylinder radius="0.03" length="0.04"/>
                 </geometry>
             </collision>
-            <xacro:inertial_cylinder mass="${mass}" length="0.04" radius="0.05">
-                <origin xyz="0 0 0" rpy="0 0 0"/>
+            <xacro:inertial_cylinder mass="${mass}" length="0.04" radius="0.03">
+                <origin xyz="0 0 -0.02" rpy="0 0 0"/>
             </xacro:inertial_cylinder>
         </link>
